File: Board/NarwhelMainV2/USB.kicad_sch (KiCad schematic)
At the start: 9 parts, among them IC8 FT232RQ-REEL, J14 USB

Commit message: Update Project MCU Board
Parts:
- removed J14: USB, library:47346-0001, symbol 47346-0001:47346-0001
- added C38: 0.1uF, Capacitor_SMD:C_0603_1608Metric_Pad1.08x0.95mm_HandSolder, symbol Device:C_Small
- added J14: USB_B_Micro, Connector_USB:USB_Micro-B_Molex_47346-0001, symbol Connector:USB_B_Micro
Connections:
- net 3.3V_USB: now also C38.2
- net D+: now also J14.3 (D+)
- net D-: now also J14.2 (D-)
- net GND: now also C38.1, J14.5 (GND), J14.6 (Shield)
- net at C34.1, FB3.1: now also J14.1 (VBUS)
Changed lines of the file:
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@@
   (junction (at 101.6 93.98) (diameter 0) (color 0 0 0 0)
   )
+  (junction (at 82.55 104.14) (diameter 0) (color 0 0 0 0)
+  )
+  (junction (at 189.23 107.95) (diameter 0) (color 0 0 0 0)
+  )
   (junction (at 200.66 107.95) (diameter 0) (color 0 0 0 0)
   )
   (junction (at 200.66 90.17) (diameter 0) (color 0 0 0 0)
   )
-  (junction (at 82.55 104.14) (diameter 0) (color 0 0 0 0)
-  )
-  (junction (at 74.93 104.14) (diameter 0) (color 0 0 0 0)
+  (junction (at 63.5 110.49) (diameter 0) (color 0 0 0 0)
   )
   (junction (at 246.38 88.9) (diameter 0) (color 0 0 0 0)
@@
   (no_connect (at 187.96 92.71))
   (no_connect (at 152.4 100.33))
-  (no_connect (at 72.39 101.6))
+  (no_connect (at 72.39 104.14))
   (no_connect (at 175.26 74.93))
   (no_connect (at 170.18 74.93))
@@
     (stroke (width 0) (type default) (color 0 0 0 0))
   )
+  (wire (pts (xy 62.23 109.22) (xy 62.23 110.49))
+    (stroke (width 0) (type default) (color 0 0 0 0))
+  )
   (wire (pts (xy 148.59 97.79) (xy 148.59 100.33))
     (stroke (width 0) (type default) (color 0 0 0 0))
   )
-  (polyline (pts (xy 46.99 76.2) (xy 46.99 114.3))
+  (polyline (pts (xy 46.99 76.2) (xy 46.99 119.38))
     (stroke (width 0) (type default) (color 0 0 0 0))
   )
@@
     (stroke (width 0) (type default) (color 0 0 0 0))
   )
+  (wire (pts (xy 189.23 125.73) (xy 189.23 129.54))
+    (stroke (width 0) (type default) (color 0 0 0 0))
+  )
   (wire (pts (xy 187.96 90.17) (xy 200.66 90.17))
     (stroke (width 0) (type default) (color 0 0 0 0))
   )
-  (wire (pts (xy 82.55 104.14) (xy 74.93 104.14))
-    (stroke (width 0) (type default) (color 0 0 0 0))
-  )
   (polyline (pts (xy 228.6 76.2) (xy 228.6 114.3))
     (stroke (width 0) (type default) (color 0 0 0 0))
@@
     (stroke (width 0) (type default) (color 0 0 0 0))
   )
+  (wire (pts (xy 189.23 107.95) (xy 200.66 107.95))
+    (stroke (width 0) (type default) (color 0 0 0 0))
+  )
   (wire (pts (xy 149.86 92.71) (xy 152.4 92.71))
     (stroke (width 0) (type default) (color 0 0 0 0))
   )
-  (wire (pts (xy 72.39 96.52) (xy 77.47 96.52))
+  (wire (pts (xy 72.39 101.6) (xy 77.47 101.6))
     (stroke (width 0) (type default) (color 0 0 0 0))
   )
@@
     (stroke (width 0) (type default) (color 0 0 0 0))
   )
-  (polyline (pts (xy 46.99 114.3) (xy 114.3 114.3))
+  (polyline (pts (xy 46.99 119.38) (xy 114.3 119.38))
     (stroke (width 0) (type default) (color 0 0 0 0))
   )
@@
     (stroke (width 0) (type default) (color 0 0 0 0))
   )
-  (wire (pts (xy 187.96 129.54) (xy 177.8 129.54))
-    (stroke (width 0) (type default) (color 0 0 0 0))
-  )
-  (wire (pts (xy 72.39 104.14) (xy 74.93 104.14))
+  (wire (pts (xy 177.8 129.54) (xy 189.23 129.54))
+    (stroke (width 0) (type default) (color 0 0 0 0))
+  )
+  (wire (pts (xy 189.23 107.95) (xy 189.23 120.65))
     (stroke (width 0) (type default) (color 0 0 0 0))
   )
@@
     (stroke (width 0) (type default) (color 0 0 0 0))
   )
-  (wire (pts (xy 74.93 104.14) (xy 74.93 106.68))
-    (stroke (width 0) (type default) (color 0 0 0 0))
-  )
   (wire (pts (xy 177.8 74.93) (xy 177.8 72.39))
     (stroke (width 0) (type default) (color 0 0 0 0))
@@
     (stroke (width 0) (type default) (color 0 0 0 0))
   )
-  (polyline (pts (xy 114.3 114.3) (xy 114.3 76.2))
+  (polyline (pts (xy 114.3 119.38) (xy 114.3 76.2))
     (stroke (width 0) (type default) (color 0 0 0 0))
   )
@@
     (stroke (width 0) (type default) (color 0 0 0 0))
   )
+  (wire (pts (xy 63.5 110.49) (xy 64.77 110.49))
+    (stroke (width 0) (type default) (color 0 0 0 0))
+  )
   (wire (pts (xy 167.64 72.39) (xy 167.64 74.93))
     (stroke (width 0) (type default) (color 0 0 0 0))
@@
     (stroke (width 0) (type default) (color 0 0 0 0))
   )
-  (wire (pts (xy 187.96 107.95) (xy 200.66 107.95))
+  (wire (pts (xy 187.96 107.95) (xy 189.23 107.95))
     (stroke (width 0) (type default) (color 0 0 0 0))
   )
@@
     (stroke (width 0) (type default) (color 0 0 0 0))
   )
+  (wire (pts (xy 63.5 110.49) (xy 63.5 111.76))
+    (stroke (width 0) (type default) (color 0 0 0 0))
+  )
   (wire (pts (xy 242.57 96.52) (xy 242.57 97.79))
     (stroke (width 0) (type default) (color 0 0 0 0))
   )
   (polyline (pts (xy 133.35 54.61) (xy 209.55 54.61))
+    (stroke (width 0) (type default) (color 0 0 0 0))
+  )
+  (wire (pts (xy 64.77 109.22) (xy 64.77 110.49))
+    (stroke (width 0) (type default) (color 0 0 0 0))
+  )
+  (wire (pts (xy 62.23 110.49) (xy 63.5 110.49))
     (stroke (width 0) (type default) (color 0 0 0 0))
   )
@@
     (effects (font (size 2 2)) (justify left bottom))
   )
-  (label "D-" (at 77.47 96.52 180)
+  (label "D-" (at 77.47 101.6 180)
     (effects (font (size 1.27 1.27)) (justify right bottom))
   )
@@
     (pin "2")
   )
+  (symbol (lib_id "Device:C_Small") (at 189.23 123.19 0) (unit 1)
+    (in_bom yes) (on_board yes) (fields_autoplaced)
+    (property "Reference" "C38" (id 0) (at 191.5541 122.2878 0)
+      (effects (font (size 1.27 1.27)) (justify left))
+    )
+    (property "Value" "0.1uF" (id 1) (at 191.5541 125.0629 0)
+      (effects (font (size 1.27 1.27)) (justify left))
+    )
+    (property "Footprint" "Capacitor_SMD:C_0603_1608Metric_Pad1.08x0.95mm_HandSolder" (id 2) (at 189.23 123.19 0)
+      (effects (font (size 1.27 1.27)) hide)
+    )
+    (property "Datasheet" "~" (id 3) (at 189.23 123.19 0)
+      (effects (font (size 1.27 1.27)) hide)
+    )
+    (pin "1")
+    (pin "2")
+  )
   (symbol (lib_id "power:+5VD") (at 190.5 102.87 270) (unit 1)
     (in_bom yes) (on_board yes)
@@
     (pin "1")
   )
-  (symbol (lib_id "47346-0001:47346-0001") (at 72.39 104.14 90) (unit 1)
-    (in_bom yes) (on_board yes)
-    (property "Reference" "J14" (id 0) (at 62.23 87.63 90)
-      (effects (font (size 1.27 1.27)) (justify left))
-    )
-    (property "Value" "USB" (id 1) (at 63.5 90.17 90)
-      (effects (font (size 1.27 1.27)) (justify left))
-    )
-    (property "Footprint" "library:47346-0001" (id 2) (at 54.61 90.17 0)
-      (effects (font (size 1.27 1.27)) (justify left) hide)
-    )
-    (property "Datasheet" "http://www.molex.com/pdm_docs/sd/473460001_sd.pdf" (id 3) (at 57.15 90.17 0)
-      (effects (font (size 1.27 1.27)) (justify left) hide)
-    )
-    (property "Description" "Micro USB B Receptacle Bottom Mount Assy Molex Right Angle SMT Type B Version 2.0 Micro USB Connector Socket, 30 V ac, 1A 47352 MICRO-USB" (id 4) (at 59.69 90.17 0)
-      (effects (font (size 1.27 1.27)) (justify left) hide)
-    )
-    (property "Height" "" (id 5) (at 62.23 90.17 0)
-      (effects (font (size 1.27 1.27)) (justify left) hide)
-    )
-    (property "Manufacturer_Name" "Molex" (id 6) (at 64.77 90.17 0)
-      (effects (font (size 1.27 1.27)) (justify left) hide)
-    )
-    (property "Manufacturer_Part_Number" "47346-0001" (id 7) (at 67.31 90.17 0)
-      (effects (font (size 1.27 1.27)) (justify left) hide)
-    )
-    (property "Mouser Part Number" "538-47346-0001" (id 8) (at 69.85 90.17 0)
-      (effects (font (size 1.27 1.27)) (justify left) hide)
-    )
-    (property "Mouser Price/Stock" "https://www.mouser.co.uk/ProductDetail/Molex/47346-0001?qs=c2CV6XM0DweJBWaSeyWeCw%3D%3D" (id 9) (at 72.39 90.17 0)
-      (effects (font (size 1.27 1.27)) (justify left) hide)
-    )
-    (property "Arrow Part Number" "" (id 10) (at 74.93 90.17 0)
-      (effects (font (size 1.27 1.27)) (justify left) hide)
-    )
-    (property "Arrow Price/Stock" "" (id 11) (at 77.47 90.17 0)
-      (effects (font (size 1.27 1.27)) (justify left) hide)
-    )
-    (pin "1")
-    (pin "2")
-    (pin "3")
-    (pin "4")
-    (pin "5")
+  (symbol (lib_id "power:GND") (at 63.5 111.76 0) (unit 1)
+    (in_bom yes) (on_board yes) (fields_autoplaced)
+    (property "Reference" "#PWR074" (id 0) (at 63.5 118.11 0)
+      (effects (font (size 1.27 1.27)) hide)
+    )
+    (property "Value" "GND" (id 1) (at 63.5 116.3225 0))
+    (property "Footprint" "" (id 2) (at 63.5 111.76 0)
+      (effects (font (size 1.27 1.27)) hide)
+    )
+    (property "Datasheet" "" (id 3) (at 63.5 111.76 0)
+      (effects (font (size 1.27 1.27)) hide)
+    )
+    (pin "1")
   )
   (symbol (lib_id "Device:C_Small") (at 82.55 99.06 0) (unit 1)
@@
     (pin "2")
   )
-  (symbol (lib_id "power:GND") (at 74.93 106.68 0) (unit 1)
-    (in_bom yes) (on_board yes) (fields_autoplaced)
-    (property "Reference" "#PWR065" (id 0) (at 74.93 113.03 0)
-      (effects (font (size 1.27 1.27)) hide)
-    )
-    (property "Value" "GND" (id 1) (at 74.93 111.2425 0))
-    (property "Footprint" "" (id 2) (at 74.93 106.68 0)
-      (effects (font (size 1.27 1.27)) hide)
-    )
-    (property "Datasheet" "" (id 3) (at 74.93 106.68 0)
+  (symbol (lib_id "power:GND") (at 82.55 104.14 0) (unit 1)
+    (in_bom yes) (on_board yes) (fields_autoplaced)
+    (property "Reference" "#PWR065" (id 0) (at 82.55 110.49 0)
+      (effects (font (size 1.27 1.27)) hide)
+    )
+    (property "Value" "GND" (id 1) (at 82.55 108.7025 0))
+    (property "Footprint" "" (id 2) (at 82.55 104.14 0)
+      (effects (font (size 1.27 1.27)) hide)
+    )
+    (property "Datasheet" "" (id 3) (at 82.55 104.14 0)
       (effects (font (size 1.27 1.27)) hide)
     )
@@
     (pin "2")
   )
+  (symbol (lib_id "Connector:USB_B_Micro") (at 64.77 99.06 0) (unit 1)
+    (in_bom yes) (on_board yes) (fields_autoplaced)
+    (property "Reference" "J14" (id 0) (at 64.77 87.4735 0))
+    (property "Value" "USB_B_Micro" (id 1) (at 64.77 90.2486 0))
+    (property "Footprint" "Connector_USB:USB_Micro-B_Molex_47346-0001" (id 2) (at 68.58 100.33 0)
+      (effects (font (size 1.27 1.27)) hide)
+    )
+    (property "Datasheet" "~" (id 3) (at 68.58 100.33 0)
+      (effects (font (size 1.27 1.27)) hide)
+    )
+    (pin "1")
+    (pin "2")
+    (pin "3")
+    (pin "4")
+    (pin "5")
+    (pin "6")
+  )
 )
