File: Board/NarwhelMainV2/EERAM.kicad_sch (KiCad schematic)
At the start: 3 parts, among them IC3 48L640T-I_SN

Commit message: Final Encoder PCB
Connections:
- net GND: now also C19.2, IC3.4 (VSS)
Changed lines of the file:
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@@
 (kicad_sch (version 20211123) (generator eeschema)
   (paper "A4")
+  (junction (at 130.81 106.68) (diameter 0) (color 0 0 0 0)
+  )
   (junction (at 181.61 99.06) (diameter 0) (color 0 0 0 0)
   )
@@
   )
   (wire (pts (xy 125.73 107.95) (xy 125.73 106.68))
+    (stroke (width 0) (type default) (color 0 0 0 0))
+  )
+  (wire (pts (xy 130.81 109.22) (xy 130.81 106.68))
     (stroke (width 0) (type default) (color 0 0 0 0))
   )
@@
     (pin "2")
   )
+  (symbol (lib_id "power:GND") (at 130.81 109.22 0) (unit 1)
+    (in_bom yes) (on_board yes) (fields_autoplaced)
+    (property "Reference" "#PWR?" (id 0) (at 130.81 115.57 0)
+      (effects (font (size 1.27 1.27)) hide)
+    )
+    (property "Value" "GND" (id 1) (at 130.81 113.7825 0))
+    (property "Footprint" "" (id 2) (at 130.81 109.22 0)
+      (effects (font (size 1.27 1.27)) hide)
+    )
+    (property "Datasheet" "" (id 3) (at 130.81 109.22 0)
+      (effects (font (size 1.27 1.27)) hide)
+    )
+    (pin "1")
+  )
   (symbol (lib_id "Device:C_Small") (at 181.61 102.87 0) (unit 1)
