File: Board/NarwhelMainV2/LVDS.kicad_sch (KiCad schematic)
At the start: 5 parts, among them IC2 SN65LVDS049PWR, J3 DS1128-09-S8B8X

Commit message: Update Board
Parts:
- added R16, R17: 300k, Resistor_SMD:R_0402_1005Metric_Pad0.72x0.64mm_HandSolder, symbol Device:R_Small
Connections:
- net +3V3: now also R16.2, R17.2
- net Rin2+: now reaches IC2.3 (RIN2+)
- net Rin2+: now also R16.1
- net Rin2-: now reaches IC2.4 (RIN2-)
- net Rin2-: now also R17.1
- no-connect marks 9 -> 7
Other:
- moved on the sheet: R15
Changed lines of the file:
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@@
   (junction (at 219.71 91.44) (diameter 0) (color 0 0 0 0)
+  )
+  (junction (at 185.42 115.57) (diameter 0) (color 0 0 0 0)
   )
   (junction (at 99.06 95.25) (diameter 0) (color 0 0 0 0)
@@
   (no_connect (at 96.52 87.63))
   (no_connect (at 205.74 86.36))
-  (no_connect (at 172.72 88.9))
-  (no_connect (at 172.72 86.36))
   (no_connect (at 73.66 95.25))
   (no_connect (at 96.52 80.01))
+  (wire (pts (xy 185.42 113.03) (xy 185.42 115.57))
+    (stroke (width 0) (type default) (color 0 0 0 0))
+  )
+  (wire (pts (xy 190.5 127) (xy 196.85 127))
+    (stroke (width 0) (type default) (color 0 0 0 0))
+  )
+  (wire (pts (xy 185.42 115.57) (xy 190.5 115.57))
+    (stroke (width 0) (type default) (color 0 0 0 0))
+  )
   (polyline (pts (xy 207.01 76.2) (xy 242.57 76.2))
     (stroke (width 0) (type default) (color 0 0 0 0))
   )
+  (wire (pts (xy 190.5 115.57) (xy 190.5 118.11))
+    (stroke (width 0) (type default) (color 0 0 0 0))
+  )
   (wire (pts (xy 219.71 91.44) (xy 229.87 91.44))
     (stroke (width 0) (type default) (color 0 0 0 0))
   )
+  (wire (pts (xy 180.34 115.57) (xy 185.42 115.57))
+    (stroke (width 0) (type default) (color 0 0 0 0))
+  )
   (wire (pts (xy 207.01 88.9) (xy 205.74 88.9))
     (stroke (width 0) (type default) (color 0 0 0 0))
@@
     (stroke (width 0) (type default) (color 0 0 0 0))
   )
+  (wire (pts (xy 180.34 118.11) (xy 180.34 115.57))
+    (stroke (width 0) (type default) (color 0 0 0 0))
+  )
+  (wire (pts (xy 180.34 127) (xy 186.69 127))
+    (stroke (width 0) (type default) (color 0 0 0 0))
+  )
+  (wire (pts (xy 180.34 123.19) (xy 180.34 127))
+    (stroke (width 0) (type default) (color 0 0 0 0))
+  )
   (wire (pts (xy 99.06 95.25) (xy 99.06 97.79))
     (stroke (width 0) (type default) (color 0 0 0 0))
@@
     (stroke (width 0) (type default) (color 0 0 0 0))
   )
+  (wire (pts (xy 190.5 123.19) (xy 190.5 127))
+    (stroke (width 0) (type default) (color 0 0 0 0))
+  )
   (wire (pts (xy 229.87 99.06) (xy 229.87 97.79))
     (stroke (width 0) (type default) (color 0 0 0 0))
   )
-  (polyline (pts (xy 156.21 63.5) (xy 156.21 113.03))
+  (polyline (pts (xy 156.21 63.5) (xy 156.21 137.16))
     (stroke (width 0) (type default) (color 0 0 0 0))
   )
@@
     (stroke (width 0) (type default) (color 0 0 0 0))
   )
-  (polyline (pts (xy 156.21 113.03) (xy 242.57 113.03))
+  (polyline (pts (xy 156.21 137.16) (xy 242.57 137.16))
     (stroke (width 0) (type default) (color 0 0 0 0))
   )
@@
     (stroke (width 0) (type default) (color 0 0 0 0))
   )
-  (polyline (pts (xy 242.57 113.03) (xy 242.57 63.5))
+  (polyline (pts (xy 242.57 137.16) (xy 242.57 63.5))
     (stroke (width 0) (type default) (color 0 0 0 0))
   )
@@
   )
   (wire (pts (xy 205.74 91.44) (xy 219.71 91.44))
+    (stroke (width 0) (type default) (color 0 0 0 0))
+  )
+  (wire (pts (xy 165.1 86.36) (xy 172.72 86.36))
+    (stroke (width 0) (type default) (color 0 0 0 0))
+  )
+  (wire (pts (xy 165.1 88.9) (xy 172.72 88.9))
     (stroke (width 0) (type default) (color 0 0 0 0))
   )
@@
     (effects (font (size 2 2)) (justify left bottom))
   )
+  (label "Rin2-" (at 165.1 88.9 0)
+    (effects (font (size 1.27 1.27)) (justify left bottom))
+  )
+  (label "Rin2+" (at 186.69 127 180)
+    (effects (font (size 1.27 1.27)) (justify right bottom))
+  )
+  (label "Rin2-" (at 196.85 127 180)
+    (effects (font (size 1.27 1.27)) (justify right bottom))
+  )
+  (label "Rin2+" (at 165.1 86.36 0)
+    (effects (font (size 1.27 1.27)) (justify left bottom))
+  )
   (global_label "SCK_D-" (shape output) (at 172.72 91.44 180) (fields_autoplaced)
     (effects (font (size 1.27 1.27)) (justify right))
@@
     )
   )
-  (global_label "MISO_D-" (shape input) (at 222.25 69.85 180) (fields_autoplaced)
-    (effects (font (size 1.27 1.27)) (justify right))
-    (property "Intersheet References" "${INTERSHEET_REFS}" (id 0) (at 211.4307 69.7706 0)
+  (global_label "MISO_D-" (shape input) (at 222.25 71.12 180) (fields_autoplaced)
+    (effects (font (size 1.27 1.27)) (justify right))
+    (property "Intersheet References" "${INTERSHEET_REFS}" (id 0) (at 211.4307 71.0406 0)
       (effects (font (size 1.27 1.27)) (justify right) hide)
     )
@@
     )
   )
-  (global_label "MISO_D+" (shape input) (at 227.33 69.85 0) (fields_autoplaced)
+  (global_label "MISO_D+" (shape input) (at 227.33 71.12 0) (fields_autoplaced)
     (effects (font (size 1.27 1.27)) (justify left))
-    (property "Intersheet References" "${INTERSHEET_REFS}" (id 0) (at 238.1493 69.9294 0)
+    (property "Intersheet References" "${INTERSHEET_REFS}" (id 0) (at 238.1493 71.1994 0)
       (effects (font (size 1.27 1.27)) (justify left) hide)
     )
@@
     (pin "MH2")
   )
+  (symbol (lib_id "Device:R_Small") (at 190.5 120.65 180) (unit 1)
+    (in_bom yes) (on_board yes) (fields_autoplaced)
+    (property "Reference" "R17" (id 0) (at 191.9986 119.7415 0)
+      (effects (font (size 1.27 1.27)) (justify right))
+    )
+    (property "Value" "300k" (id 1) (at 191.9986 122.5166 0)
+      (effects (font (size 1.27 1.27)) (justify right))
+    )
+    (property "Footprint" "Resistor_SMD:R_0402_1005Metric_Pad0.72x0.64mm_HandSolder" (id 2) (at 190.5 120.65 0)
+      (effects (font (size 1.27 1.27)) hide)
+    )
+    (property "Datasheet" "~" (id 3) (at 190.5 120.65 0)
+      (effects (font (size 1.27 1.27)) hide)
+    )
+    (pin "1")
+    (pin "2")
+  )
   (symbol (lib_id "power:GND") (at 219.71 100.33 0) (unit 1)
     (in_bom yes) (on_board yes) (fields_autoplaced)
@@
     (pin "1")
   )
-  (symbol (lib_id "Device:R_Small") (at 224.79 69.85 90) (unit 1)
-    (in_bom yes) (on_board yes) (fields_autoplaced)
-    (property "Reference" "R15" (id 0) (at 224.79 65.1469 90))
-    (property "Value" "100r" (id 1) (at 224.79 67.922 90))
-    (property "Footprint" "Resistor_SMD:R_0603_1608Metric_Pad0.98x0.95mm_HandSolder" (id 2) (at 224.79 69.85 0)
-      (effects (font (size 1.27 1.27)) hide)
-    )
-    (property "Datasheet" "~" (id 3) (at 224.79 69.85 0)
+  (symbol (lib_id "Device:R_Small") (at 224.79 71.12 90) (unit 1)
+    (in_bom yes) (on_board yes) (fields_autoplaced)
+    (property "Reference" "R15" (id 0) (at 224.79 66.4169 90))
+    (property "Value" "100r" (id 1) (at 224.79 69.192 90))
+    (property "Footprint" "Resistor_SMD:R_0603_1608Metric_Pad0.98x0.95mm_HandSolder" (id 2) (at 224.79 71.12 0)
+      (effects (font (size 1.27 1.27)) hide)
+    )
+    (property "Datasheet" "~" (id 3) (at 224.79 71.12 0)
       (effects (font (size 1.27 1.27)) hide)
     )
@@
     (pin "9")
   )
+  (symbol (lib_id "Device:R_Small") (at 180.34 120.65 180) (unit 1)
+    (in_bom yes) (on_board yes) (fields_autoplaced)
+    (property "Reference" "R16" (id 0) (at 181.8386 119.7415 0)
+      (effects (font (size 1.27 1.27)) (justify right))
+    )
+    (property "Value" "300k" (id 1) (at 181.8386 122.5166 0)
+      (effects (font (size 1.27 1.27)) (justify right))
+    )
+    (property "Footprint" "Resistor_SMD:R_0402_1005Metric_Pad0.72x0.64mm_HandSolder" (id 2) (at 180.34 120.65 0)
+      (effects (font (size 1.27 1.27)) hide)
+    )
+    (property "Datasheet" "~" (id 3) (at 180.34 120.65 0)
+      (effects (font (size 1.27 1.27)) hide)
+    )
+    (pin "1")
+    (pin "2")
+  )
   (symbol (lib_id "power:+3.3V") (at 219.71 91.44 0) (unit 1)
     (in_bom yes) (on_board yes) (fields_autoplaced)
@@
       (effects (font (size 1.27 1.27)) hide)
     )
+    (pin "1")
+  )
+  (symbol (lib_id "power:+3.3V") (at 185.42 113.03 0) (unit 1)
+    (in_bom yes) (on_board yes) (fields_autoplaced)
+    (property "Reference" "#PWR075" (id 0) (at 185.42 116.84 0)
+      (effects (font (size 1.27 1.27)) hide)
+    )
+    (property "Value" "+3.3V" (id 1) (at 185.42 109.4255 0))
+    (property "Footprint" "" (id 2) (at 185.42 113.03 0)
+      (effects (font (size 1.27 1.27)) hide)
+    )
+    (property "Datasheet" "" (id 3) (at 185.42 113.03 0)
+      (effects (font (size 1.27 1.27)) hide)
+    )
