File: Board/NarwhelMainV2/MCU.kicad_sch (KiCad schematic)
At the start: 42 parts, among them IC1 STM32H733VGT6, J1 Pinheader 3P, J16 HX_6p, J2 Pinheader 2*4, J5 Pinheader 4p, SW1 SW_Push, Y1 25MHz

Commit message: Update Board
Parts:
- C14: value 6nF -> 0.1uF
Changed lines of the file:
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@@
       (effects (font (size 1.27 1.27)) (justify left))
     )
-    (property "Value" "6nF" (id 1) (at 144.78 102.87 0)
+    (property "Value" "0.1uF" (id 1) (at 144.78 102.87 0)
       (effects (font (size 1.27 1.27)) (justify left))
     )
