File: Board/NarwhelMainV2/NarwhelMainV2.kicad_pcb (KiCad board)
At the start: 4 copper layers, 100 x 100 mm, 107 parts, among them IC1 STM32H733VGT6, IC2 SN65LVDS049PWR, IC3 48L640T-I_SN, IC4 TPS2400DBVT, IC5 LD39100PU33RY, IC6 TMP75CQDRQ1, IC7 TMP75CQDRQ1, IC8 FT232RQ-REEL, J1 Pinheader 3P, J10 HX_3p, J11 HX_3p, J12 HX_3p, J13 HX_3p, J14 USB, J15 Conn_01x04_Male, J16 HX_6p, J2 Pinheader 2*4, J3 DS1128-09-S8B8X, J4 Screw_Terminal_16p, J5 Pinheader 4p, J6 Screw_Terminal_2P, J7 Pinheader 3P, J8 HX_3p, J9 HX_3p, Q1 BSZ42DN25NS3_G, Q2 AO3401A, SW1 SW_Push, U1 TXS0108EPW, U2 TXS0108EPW, U3 AMS1117CD-5.0, Y1 25MHz

Commit message: Update Project MCU Board
Parts:
- added C38: 0.1uF, Capacitor_SMD:C_0603_1608Metric_Pad1.08x0.95mm_HandSolder, F.Cu at (180.4, 134.0)
- added REF**: KiCad-Logo2_5mm_SilkScreen, Symbol:KiCad-Logo2_5mm_SilkScreen, F.Cu at (164.0, 134.0)
- J14: value USB -> USB_B_Micro; footprint library:47346-0001 -> Connector_USB:USB_Micro-B_Molex_47346-0001
- moved C37 3.41 mm to (182.8, 114.2)
- moved IC7 3.41 mm to (186.6, 116.0)
- moved R12 3.13 mm to (160.9, 115.8), turned to 180 degrees
- moved R11 2.77 mm to (160.9, 118.8), turned to 180 degrees
- moved J14 2.54 mm to (178.2, 142.4), turned to 180 degrees
- moved C36 0.40 mm to (115.2, 71.2)
Connections:
- J14 pad 6: (no net) -> GND
Routing:
- net /Microcontroller/SCL: track 0.00 -> 189.1 mm, vias 0 -> 3
- net /Microcontroller/SDA: track 0.00 -> 187.4 mm, vias 0 -> 3
- net /UART_to_USB/3.3V_USB: track 0.00 -> 31.7 mm, vias 0 -> 3
- net GND: track 107.6 -> 115.0 mm, vias 76 -> 143
- net +3V3: track 102.7 -> 107.1 mm, vias 28 -> 32
- net +5VD: track 191.4 -> 189.9 mm
- net Net-(C34-Pad1): track 4.92 -> 6.30 mm, vias 6 -> 4
- net /UART_to_USB/D+: track 8.78 -> 9.59 mm
- net /UART_to_USB/D-: track 8.76 -> 9.57 mm
- net /Microcontroller/RX: track 30.6 -> 30.0 mm
Other:
- board text added: "Design By"
- board text added: "Thansak Pongpaket"

Commit message: Final Encoder PCB
Connections:
- C19 pad 2: Net-(C19-Pad2) -> GND
- IC3 pad 4: Net-(C19-Pad2) -> GND
Routing:
- net Net-(C19-Pad2): track 4.46 -> 0.00 mm
- net GND: track 115.0 -> 119.4 mm, vias 143 -> 145
- net /Microcontroller/ENC_TImer3A: track 82.8 -> 85.1 mm

Commit message: Update Board
Parts:
- added R16: 300k, Resistor_SMD:R_0402_1005Metric_Pad0.72x0.64mm_HandSolder, F.Cu at (179.8, 82.5)
- added R17: 300k, Resistor_SMD:R_0402_1005Metric_Pad0.72x0.64mm_HandSolder, F.Cu at (179.8, 81.2)
- C14: value 6nF -> 0.1uF
- moved G*** 1.67 mm to (187.9, 95.3)
Connections:
- IC2 pad 3: unconnected-(IC2-Pad3) -> /Low-Voltage Differential Signal/Rin2+
- IC2 pad 4: unconnected-(IC2-Pad4) -> /Low-Voltage Differential Signal/Rin2-
Routing:
- net GND: track 119.4 -> 111.7 mm, vias 145 -> 142
- net /Low-Voltage Differential Signal/Rin2+: track 0.00 -> 4.32 mm
- net /Low-Voltage Differential Signal/Rin2-: track 0.00 -> 4.12 mm
- net +3V3: track 107.1 -> 109.6 mm, vias 32 -> 33
Other:
- board text added: "+"
- board text added: "23/1/22"
- board text added: "Base Encoder"
- board text added: "CS Encoder"
- board text added: "DIR1"
- board text added: "DIR2"
- board text added: "DIR3"
- board text added: "DIR4"
- board text added: "DIR5"
- board text added: "EMSw"
- board text added: "EN123"
- board text added: "EN45"
- board text added: "Griper0"
- board text added: "Griper1"
- board text added: "Griper2"
- board text added: "Module 8-9 G.3"
- board text added: "Power Encoder"
- board text added: "Power Supply"
- board text added: "STEP1"
- board text added: "STEP2"
- board text added: "STEP3"
- board text added: "STEP4"
- board text added: "STEP5"
- board text added: "Temp Sensor"
