File: Board/NarWhelEncoderV2/NarWhelEncoderV2.kicad_pcb (KiCad board)
At the start: 4 copper layers, 58 x 45 mm, 36 parts, among them IC1 AS5047U-HTSM, IC2 SN65LVDS049PWR, IC3 LM1117-3.3, J1 HX_3p, J2 DS1128-09-S8B8X, J3 DS1128-09-S8B8X, Q1 2N7002, Q2 2N7002

Commit message: Update Board
Routing:
- net +3V3: track 6.74 -> 12.9 mm, vias 6 -> 7
- net GND: vias 24 -> 27
Changed lines of the file:
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@@
       (outputformat 1)
       (mirror false)
-      (drillshape 1)
+      (drillshape 0)
       (scaleselection 1)
-      (outputdirectory "")
+      (outputdirectory "Gerber/")
     )
   )
@@
     (fp_line (start -2.45 2.35) (end -2.45 -3.4) (layer "B.Fab") (width 0.1))
     (fp_line (start -2.45 -3.4) (end 7.45 -3.4) (layer "B.Fab") (width 0.1))
-    (pad "1" thru_hole roundrect locked (at 0 0 180) (size 1.7 1.95) (drill 0.95) (layers *.Cu *.Mask) (roundrect_rratio 0.147059)
+    (pad "1" thru_hole roundrect locked (at 0 0 180) (size 1.7 1.95) (drill 0.95) (layers *.Cu *.Mask) (roundrect_rratio 0.1470588235)
       (net 1 "/Vin") (pinfunction "Pin_1") (pintype "passive"))
     (pad "2" thru_hole oval locked (at 2.5 0 180) (size 1.7 1.95) (drill 0.95) (layers *.Cu *.Mask)
@@
   (via (at 168.1 118.2) (size 0.6) (drill 0.3) (layers "F.Cu" "B.Cu") (net 2))
   (via (at 175 115) (size 0.6) (drill 0.3) (layers "F.Cu" "B.Cu") (net 2))
+  (via (at 152.2 112.4) (size 0.6) (drill 0.3) (layers "F.Cu" "B.Cu") (free) (net 2))
   (via (at 173.85 107.95) (size 0.8) (drill 0.4) (layers "F.Cu" "B.Cu") (net 2))
   (via (at 164 107.5) (size 0.8) (drill 0.4) (layers "F.Cu" "B.Cu") (free) (net 2))
@@
   (via (at 162.9 107.5) (size 0.8) (drill 0.4) (layers "F.Cu" "B.Cu") (free) (net 2))
   (via (at 180.2 119.9) (size 0.6) (drill 0.3) (layers "F.Cu" "B.Cu") (free) (net 2))
+  (via (at 147.4 117.3) (size 0.6) (drill 0.3) (layers "F.Cu" "B.Cu") (free) (net 2))
   (via (at 160.3 120.4) (size 0.6) (drill 0.3) (layers "F.Cu" "B.Cu") (net 2))
   (via (at 171.9 126.8) (size 0.6) (drill 0.3) (layers "F.Cu" "B.Cu") (net 2))
@@
   (via (at 165 107.5) (size 0.8) (drill 0.4) (layers "F.Cu" "B.Cu") (free) (net 2))
   (via (at 147.9 132.5) (size 0.6) (drill 0.3) (layers "F.Cu" "B.Cu") (free) (net 2))
+  (via (at 152.4 116.4) (size 0.6) (drill 0.3) (layers "F.Cu" "B.Cu") (free) (net 2))
   (via (at 162.9 106.3) (size 0.8) (drill 0.4) (layers "F.Cu" "B.Cu") (free) (net 2))
   (via (at 159.1 118.5) (size 0.6) (drill 0.3) (layers "F.Cu" "B.Cu") (net 2))
@@
   (segment (start 162.3375 119.25) (end 162.2 119.1125) (width 0.25) (layer "F.Cu") (net 3))
   (segment (start 174 117.5) (end 172.688 117.5) (width 0.25) (layer "F.Cu") (net 3))
+  (segment (start 159.5 124.2) (end 159.5 124) (width 0.25) (layer "F.Cu") (net 3))
+  (segment (start 154.6625 124.35) (end 159.65 124.35) (width 0.25) (layer "F.Cu") (net 3))
   (segment (start 162.2 119.1125) (end 162.2 118.4) (width 0.25) (layer "F.Cu") (net 3))
+  (segment (start 162.2375 119.25) (end 162.2375 119.9625) (width 0.25) (layer "F.Cu") (net 3))
   (segment (start 160.338 117.825) (end 162.2 117.825) (width 0.25) (layer "F.Cu") (net 3))
+  (segment (start 159.65 124.35) (end 159.5 124.2) (width 0.25) (layer "F.Cu") (net 3))
   (segment (start 174.2125 117.7125) (end 174 117.5) (width 0.25) (layer "F.Cu") (net 3))
   (segment (start 175 117.7125) (end 174.2125 117.7125) (width 0.25) (layer "F.Cu") (net 3))
+  (segment (start 162.2375 119.9625) (end 162.2 120) (width 0.25) (layer "F.Cu") (net 3))
   (via (at 160 123.5) (size 0.6) (drill 0.3) (layers "F.Cu" "B.Cu") (free) (net 3))
   (via (at 160 124.5) (size 0.6) (drill 0.3) (layers "F.Cu" "B.Cu") (free) (net 3))
+  (via (at 162.2 120) (size 0.6) (drill 0.3) (layers "F.Cu" "B.Cu") (net 3))
   (via (at 160.5 124) (size 0.6) (drill 0.3) (layers "F.Cu" "B.Cu") (free) (net 3))
   (via (at 162.2 118.4) (size 0.6) (drill 0.3) (layers "F.Cu" "B.Cu") (net 3))
@@
     )
   )
+  (zone (net 2) (net_name "GND") (layer "F.Cu") (hatch edge 0.508)
+    (connect_pads (clearance 0))
+    (min_thickness 0.254) (filled_areas_thickness no)
+    (fill yes (thermal_gap 0.508) (thermal_bridge_width 0.508))
+    (polygon
+      (pts
+        (xy 157.4 140)
+        (xy 135 139.9)
+        (xy 135 95)
+        (xy 157.4 95)
+      )
+    )
+  )
   (zone (net 0) (net_name "") (layer "F.Cu") (hatch edge 0.508)
     (connect_pads (clearance 0))
@@
       (pts
         (xy 195 140)
-        (xy 135 140)
-        (xy 135 95)
+        (xy 157.6 140)
+        (xy 157.6 95)
         (xy 195 95)
       )
